Commit message: Made various improvements.

File: ackermann_vehicle_description/urdf/em_3905.urdf.xacro (robot description, xacro)
@@ -59,6 +59,6 @@
   <xacro:property name="wheel_travel" value="0.084"/>
   <xacro:property name="shock_z_offset" value="0.0655"/>
+<!--
   <xacro:property name="shock_stroke" value="0.028575"/>
-<!--
   <xacro:property name="shock_spring_constant" value="437.817"/>
   <xacro:property name="shock_damping" value="36.2416"/>
@@ -67,7 +67,7 @@
        no_load_speed is measured in rad/s. stall_torque is measured in
        N m. kp is stall_torque / (pi / 4). -->
-<!--
   <xacro:property name="no_load_speed" value="4.553"/>
   <xacro:property name="stall_torque" value="0.5649"/>
+<!--
   <xacro:property name="kp" value="0.7193"/>
   <xacro:property name="ki" value="0"/>
@@ -76,4 +76,7 @@
   <xacro:property name="i_max" value="0"/>
 -->
+  <!-- ctrl_period is the control period for the ros_control plug-in. It is
+       measured in seconds. -->
+  <xacro:property name="ctrl_period" value="0.001"/>
   <material name="battery_mat">
     <color rgba="0 0 1 1"/>
@@ -248,6 +251,8 @@
       <child link="${lr_prefix}_${fr_prefix}_axle_carrier"/>
       <axis xyz="0 0 -1"/>
+      <!-- stall_torque is multiplied by two because steering is controlled by
+           two servos connected in parallel. -->
       <limit lower="${-degrees_45}" upper="${degrees_45}"
-             effort="1000" velocity="1000"/>
+             effort="${2 * stall_torque}" velocity="${no_load_speed}"/>
     </joint>
     <transmission name="${lr_prefix}_steering_trans"
@@ -327,5 +332,5 @@
       <robotNamespace>/</robotNamespace>
       <robotParam>robot_description</robotParam>
-      <controlPeriod>0.001</controlPeriod>
+      <controlPeriod>${ctrl_period}</controlPeriod>
     </plugin>
   </gazebo>

Commit message: Removed unused elements. Positive steering angles now cause the front wheels to rotate to the left. Positive shock absorber position values now cause the shocks to extend, moving the wheels downward.

File: ackermann_vehicle_description/urdf/em_3905.urdf.xacro (robot description, xacro)
@@ -4,5 +4,5 @@
 truck.
 Lengths are measured in meters, angles are measured in radians, and masses are
-measured in kilograms.
+measured in kilograms. All of these values are approximations.
 To work with Gazebo, each link must have an inertial element, even if
 the link only serves to connect two joints. To be visible in Gazebo, a link
@@ -60,8 +60,5 @@
        the shock absorbers are fully extended. axle_length is the distance
        from a U joint to the corresponding hex hub. wheel_travel is the
-       vertical wheel travel. shock_spring_constant is the constant of an
-       TODO Ultra Shock spring, measured in N/m. shock_damping is the shock
-       absorber's viscous damping coefficient, measured in Ns/m. Its value is
-       sqrt(3 * shock_spring_constant). -->
+       vertical wheel travel. -->
   <xacro:property name="wheelbase" value="0.335"/>
   <xacro:property name="hex_hub_dist" value="0.365"/>
@@ -69,21 +66,9 @@
   <xacro:property name="wheel_travel" value="0.084"/>
   <xacro:property name="shock_z_offset" value="0.0655"/>
-<!--
-  <xacro:property name="shock_stroke" value="0.028575"/>
-  <xacro:property name="shock_spring_constant" value="437.817"/>
-  <xacro:property name="shock_damping" value="36.2416"/>
--->
   <!-- These constants are used to simulate a Traxxas 2056 servo operated at
        6 V. no_load_speed is measured in rad/s. stall_torque is measured in
-       N m. kp is stall_torque / (pi / 4). -->
+       N m. -->
   <xacro:property name="no_load_speed" value="4.553"/>
   <xacro:property name="stall_torque" value="0.5649"/>
-<!--
-  <xacro:property name="kp" value="0.7193"/>
-  <xacro:property name="ki" value="0"/>
-  <xacro:property name="kd" value="0.0001"/>
-  <xacro:property name="i_min" value="0"/>
-  <xacro:property name="i_max" value="0"/>
--->
   <!-- ctrl_period is the control period for the ros_control plug-in. It is
        measured in seconds. -->
@@ -188,5 +173,5 @@
                    ${lr_reflect * ((hex_hub_dist / 2) - axle_length)}
                    ${(wheel_travel / 2) - shock_z_offset}"/>
-      <axis xyz="0 0 1"/>
+      <axis xyz="0 0 -1"/>
       <limit lower="${-wheel_travel / 2}" upper="${wheel_travel / 2}"
              effort="1000" velocity="1000"/>
@@ -212,4 +197,5 @@
       <origin rpy="${degrees_90} 0 0"/>
       <axis xyz="0 0 -1"/>
+      <limit effort="1000" velocity="1000"/>
     </joint>
     <transmission name="${lr_prefix}_${fr_prefix}_axle_trans">
@@ -260,9 +246,7 @@
       <parent link="${lr_prefix}_steering_link"/>
       <child link="${lr_prefix}_${fr_prefix}_axle_carrier"/>
-      <axis xyz="0 0 -1"/>
-      <!-- stall_torque is multiplied by two because steering is controlled by
-           two servos connected in parallel. -->
+      <axis xyz="0 0 1"/>
       <limit lower="${-degrees_45}" upper="${degrees_45}"
-             effort="${2 * stall_torque}" velocity="${no_load_speed}"/>
+             effort="${stall_torque}" velocity="${no_load_speed}"/>
     </joint>
     <transmission name="${lr_prefix}_steering_trans">
@@ -345,45 +329,3 @@
     </plugin>
   </gazebo>
-<!--
-    <gazebo>
-      <controller:gazebo_ros_spring name="${lr_prefix}_${fr_prefix}_spring" plugin="libgazebo_ros_spring.so">
-        <alwaysOn>true</alwaysOn>
-        <updateRate>1000</updateRate>
-        <jointName>${lr_prefix}_${fr_prefix}_shock</jointName>
-        <springConstant>${2 * (shock_stroke * shock_spring_constant /
-          wheel_travel)}</springConstant>
-        <equilibriumPosition>${-wheel_travel / 2}</equilibriumPosition>
-        <dampingCoefficient>${2 * shock_damping}</dampingCoefficient>
-      </controller:gazebo_ros_spring>
-    </gazebo>
--->
-    <!-- Steering controller -->
-<!--
-    <controller:ackermann_steering_controller name="steering_controller" plugin="libackermann_steering_controller.so">
-      <alwaysOn>true</alwaysOn>
-      <updateRate>1000</updateRate>
-      <leftJointName>left_steering_joint</leftJointName>
-      <rightJointName>right_steering_joint</rightJointName>
-      <jointDistance>${hex_hub_dist - 2 * axle_length}</jointDistance>
-      <wheelbase>${wheelbase}</wheelbase>
--->
-      <!-- stallTorque is multiplied by two because steering is controlled by
-           two servos connected in parallel. -->
-<!--
-      <noLoadSpeed>${no_load_speed}</noLoadSpeed>
-      <stallTorque>${2 * stall_torque}</stallTorque>
-      <kP>${kp}</kP>
-      <kI>${ki}</kI>
-      <kD>${kd}</kD>
-      <iMin>${i_min}</iMin>
-      <iMax>${i_max}</iMax>
-    </controller:ackermann_steering_controller>
--->
-    <!-- ESC -->
-<!--
-    <controller:electronic_speed_control name="esc" plugin="libelectronic_speed_control.so">
-      <alwaysOn>true</alwaysOn>
-      <updateRate>1000</updateRate>
-    </controller:electronic_speed_control>
--->
 </robot>

Commit message: Changed joint effort and velocity limits.

File: ackermann_vehicle_description/urdf/em_3905.urdf.xacro (robot description, xacro)
@@ -9,9 +9,11 @@
 must have a collision element. Furthermore, the link must have a Gazebo
 material.
-Traxxas(R) and E-Maxx(R) are registered trademarks of Traxxas Management, LLC.
-em_3905.urdf.xacro was independently created by Wunderkammer Laboratory, and
-neither em_3905.urdf.xacro nor Wunderkammer Laboratory is affiliated with,
-sponsored by, approved by, or endorsed by Traxxas Management, LLC. All other
-trademarks and service marks are the property of their respective owners.
+Traxxas(R), E-Maxx(R), and Titan(R) are registered trademarks of Traxxas
+Management, LLC. em_3905.urdf.xacro was independently created by Wunderkammer
+Laboratory, and neither em_3905.urdf.xacro nor Wunderkammer Laboratory is
+affiliated with, sponsored by, approved by, or endorsed by Traxxas Management,
+LLC. Mabuchi Motor(R) is a registered trademark of Mabuchi Motor Co., Ltd.
+Corporation Japan. All other trademarks and service marks are the property of
+their respective owners.
 Copyright (c) 2011-2013 Wunderkammer Laboratory
 Licensed under the Apache License, Version 2.0 (the "License");
@@ -51,5 +53,5 @@
        inset from the outer edge of the tire. It is set so that each wheel
        is a "zero offset" wheel. hex_hub_depth = tire_width / 2 -
-       axle_length. xacro cannot compute hex_hub_depth's value. -->
+       axle_length. -->
   <xacro:property name="hub_dia" value="0.09652"/>
   <xacro:property name="tire_dia" value="0.14605"/>
@@ -66,12 +68,29 @@
   <xacro:property name="wheel_travel" value="0.084"/>
   <xacro:property name="shock_z_offset" value="0.0655"/>
+  <!-- shock_eff_limit is 2 * ((shock_stroke / 2) * shock_spring_constant) N.
+       shock_stroke is 0.028575 meters. shock_spring_constant, an approximation
+       of a Traxxas Ultra Shock shock absorber spring's constant, is
+       437.817 N/m. -->
+  <xacro:property name="shock_eff_limit" value="12.5106"/>
+  <xacro:property name="shock_vel_limit" value="1000"/>
+  <!-- The specifications for a Titan(R) 550 motor could not be found, so the
+       stall torque of a Mabuchi Motor(R) RS-550VC-7525 motor was used instead.
+       num_spur_gear_teeth = 68
+       num_pinion_gear_teeth = 19
+       final_gear_ratio = (num_spur_gear_teeth / num_pinion_gear_teeth) *
+         5.22 = 18.68
+       stall_torque = 0.549 N m
+       axle_eff_limit = ((2 * stall_torque) * final_gear_ratio) / 4 =
+         5.12766 N m
+       max_speed = 40 mph (30+ mph) = 17.8816 m/s
+       axle_vel_limit = (2 * pi) * (max_speed / (pi * tire_dia)) =
+         244.8696 rad/s -->
+  <xacro:property name="axle_eff_limit" value="5.12766"/>
+  <xacro:property name="axle_vel_limit" value="244.8696"/>
   <!-- These constants are used to simulate a Traxxas 2056 servo operated at
-       6 V. no_load_speed is measured in rad/s. stall_torque is measured in
-       N m. -->
-  <xacro:property name="no_load_speed" value="4.553"/>
-  <xacro:property name="stall_torque" value="0.5649"/>
-  <!-- ctrl_period is the control period for the ros_control plug-in. It is
-       measured in seconds. -->
-  <xacro:property name="ctrl_period" value="0.001"/>
+       6 V. servo_stall_torque is measured in N m. servo_no_load_speed is
+       measured in rad/s. -->
+  <xacro:property name="servo_stall_torque" value="0.5649"/>
+  <xacro:property name="servo_no_load_speed" value="4.553"/>
   <material name="battery_mat">
     <color rgba="0 0 1 1"/>
@@ -175,5 +194,5 @@
       <axis xyz="0 0 -1"/>
       <limit lower="${-wheel_travel / 2}" upper="${wheel_travel / 2}"
-             effort="1000" velocity="1000"/>
+             effort="${shock_eff_limit}" velocity="${shock_vel_limit}"/>
     </joint>
     <transmission name="${lr_prefix}_${fr_prefix}_shock_trans">
@@ -182,4 +201,5 @@
       <actuator name="${lr_prefix}_${fr_prefix}_shock_act">
         <hardwareInterface>EffortJointInterface</hardwareInterface>
+        <mechanicalReduction>1</mechanicalReduction>
       </actuator>
     </transmission>
@@ -197,5 +217,5 @@
       <origin rpy="${degrees_90} 0 0"/>
       <axis xyz="0 0 -1"/>
-      <limit effort="1000" velocity="1000"/>
+      <limit effort="${axle_eff_limit}" velocity="${axle_vel_limit}"/>
     </joint>
     <transmission name="${lr_prefix}_${fr_prefix}_axle_trans">
@@ -204,4 +224,5 @@
       <actuator name="${lr_prefix}_${fr_prefix}_axle_act">
         <hardwareInterface>EffortJointInterface</hardwareInterface>
+        <mechanicalReduction>1</mechanicalReduction>
       </actuator>
     </transmission>
@@ -248,5 +269,5 @@
       <axis xyz="0 0 1"/>
       <limit lower="${-degrees_45}" upper="${degrees_45}"
-             effort="${stall_torque}" velocity="${no_load_speed}"/>
+             effort="${servo_stall_torque}" velocity="${servo_no_load_speed}"/>
     </joint>
     <transmission name="${lr_prefix}_steering_trans">
@@ -255,4 +276,5 @@
       <actuator name="${lr_prefix}_steering_act">
         <hardwareInterface>EffortJointInterface</hardwareInterface>
+        <mechanicalReduction>1</mechanicalReduction>
       </actuator>
     </transmission>
@@ -298,6 +320,6 @@
     </collision>
     <xacro:solid_cuboid_inertial
-       width="${chassis_length}" depth="${chassis_width}"
-       height="${chassis_height}" mass="${chassis_mass}">
+        width="${chassis_length}" depth="${chassis_width}"
+        height="${chassis_height}" mass="${chassis_mass}">
       <origin xyz="0 0 ${-chassis_height / 2}"/>
     </xacro:solid_cuboid_inertial>
@@ -307,6 +329,6 @@
   </gazebo>
   <joint name="base_link_to_chasis" type="fixed">
-      <parent link="base_link"/>
-      <child link="chassis"/>
+    <parent link="base_link"/>
+    <child link="chassis"/>
   </joint>
   <!-- Batteries -->
@@ -323,9 +345,5 @@
                     lr_reflect="-1" fr_reflect="-1"/>
   <gazebo>
-    <plugin name="ros_control" filename="libgazebo_ros_control.so">
-      <robotNamespace>/</robotNamespace>
-      <robotParam>robot_description</robotParam>
-      <controlPeriod>${ctrl_period}</controlPeriod>
-    </plugin>
+    <plugin name="ros_control" filename="libgazebo_ros_control.so"/>
   </gazebo>
 </robot>

Commit message: Added the ctrl_period property.

File: ackermann_vehicle_description/urdf/em_3905.urdf.xacro (robot description, xacro)
@@ -93,4 +93,6 @@
   <xacro:property name="servo_stall_torque" value="0.5649"/>
   <xacro:property name="servo_no_load_speed" value="4.553"/>
+  <!-- ctrl_period is gazebo_ros_control's control period. Unit: hertz. -->
+  <xacro:property name="ctrl_period" value="0.01"/>
   <material name="battery_mat">
     <color rgba="0 0 1 1"/>
@@ -345,5 +347,11 @@
                     lr_reflect="-1" fr_reflect="-1"/>
   <gazebo>
-    <plugin name="ros_control" filename="libgazebo_ros_control.so"/>
+    <plugin name="gazebo_ros_control" filename="libgazebo_ros_control.so">
+      <!-- As of 10/7/13, setting controlPeriod to a value greater than
+           Gazebo's simulation period prevents the shock absorbers from
+           working.
+      <controlPeriod>${ctrl_period}</controlPeriod>
+      -->
+    </plugin>
   </gazebo>
 </robot>

Commit message: Removed the ctrl_period property.

File: ackermann_vehicle_description/urdf/em_3905.urdf.xacro (robot description, xacro)
@@ -16,5 +16,5 @@
 Corporation Japan. All other trademarks and service marks are the property of
 their respective owners.
-Copyright (c) 2011-2013 Wunderkammer Laboratory
+Copyright (c) 2011-2014 Wunderkammer Laboratory
 Licensed under the Apache License, Version 2.0 (the "License");
 you may not use this file except in compliance with the License.
@@ -93,6 +93,4 @@
   <xacro:property name="servo_stall_torque" value="0.5649"/>
   <xacro:property name="servo_no_load_speed" value="4.553"/>
-  <!-- ctrl_period is gazebo_ros_control's control period. Unit: hertz. -->
-  <xacro:property name="ctrl_period" value="0.01"/>
   <material name="battery_mat">
     <color rgba="0 0 1 1"/>
@@ -347,11 +345,5 @@
                     lr_reflect="-1" fr_reflect="-1"/>
   <gazebo>
-    <plugin name="gazebo_ros_control" filename="libgazebo_ros_control.so">
-      <!-- As of 10/7/13, setting controlPeriod to a value greater than
-           Gazebo's simulation period prevents the shock absorbers from
-           working.
-      <controlPeriod>${ctrl_period}</controlPeriod>
-      -->
-    </plugin>
+    <plugin name="gazebo_ros_control" filename="libgazebo_ros_control.so"/>
   </gazebo>
 </robot>

Commit message: Fixed joint name to coincide with link names

File: ackermann_vehicle_description/urdf/em_3905.urdf.xacro (robot description, xacro)
@@ -340,5 +340,5 @@
     <material>Gazebo/Grey</material>
   </gazebo>
-  <joint name="base_link_to_chasis" type="fixed">
+  <joint name="base_link_to_chassis" type="fixed">
     <parent link="base_link"/>
     <child link="chassis"/>
