Commit message: Added hokuyo utm30lx model and Added dependency hector_models in  package.xml

File: ackermann_vehicle_description/urdf/em_3905_hokuyo.urdf.xacro (robot description, xacro)
@@ -28,6 +28,6 @@
 -->
 <robot name="em_3905" xmlns:xacro="http://www.ros.org/wiki/xacro">
+  <xacro:include filename="$(find hector_sensors_description)/urdf/hokuyo_utm30lx.urdf.xacro"/>
   <!-- Degree-to-radian conversions -->
-  <!--xacro:include filename="$(find hector_sensors_description)/urdf/hokuyo_utm30lx.urdf.xacro"/-->
   <xacro:property name="degrees_45" value="0.785398163"/>
   <xacro:property name="degrees_90" value="1.57079633"/>
@@ -358,5 +358,5 @@
                     lr_reflect="-1" fr_reflect="-1"/>
   <!-- LiDAR -->
-  <link name="hokuyo_link">
+  <!-- <link name="hokuyo_link">
     <visual>
       <geometry>
@@ -378,10 +378,10 @@
   <gazebo>
     <plugin name="gazebo_ros_control" filename="libgazebo_ros_control.so"/>
-  </gazebo>
-  <!--hokuyo_utm30lx_model name="hokuyo_laser" parent="base_link">
-    <origin xyz="0 0 +0.30" rpy="0 0 0" />
-  </hokuyo_utm30lx_model-->
+  </gazebo> -->
+  <xacro:hokuyo_utm30lx_model name="hokuyo_laser" parent="base_link">
+    <origin xyz="0 0 0.11" rpy="0 0 0" />
+  </xacro:hokuyo_utm30lx_model>
   <xacro:macro name="hokuyo_laser">
-    <gazebo reference="hokuyo_link">
+    <gazebo reference="hokuyo_laser_frame">
       <sensor type="gpu_ray" name="hokuyo_laser">
         <pose>0 0 0 0 0 0</pose>
