Commit message: Added imu sensor

File: ackermann_vehicle_description/urdf/em_3905_hokuyo_imu.urdf.xacro (robot description, xacro)
@@ -376,5 +376,5 @@
     <child link="hokuyo_link" />
   </joint>
- -->
+-->
   <gazebo>
     <plugin name="gazebo_ros_control" filename="libgazebo_ros_control.so"/>
@@ -421,3 +421,41 @@
   </xacro:macro>
   <xacro:hokuyo_laser/>
+  <!-- IMU frame -->
+  <link name="imu_link">
+    <visual>
+      <geometry>
+        <box size="0.02 0.035 0.002"/>
+      </geometry>
+      <material name="Green"/>
+    </visual>
+    <inertial>
+      <mass value="0.001"/>
+      <origin xyz="0 0 0"/>
+      <inertia ixx="0.0001" ixy="0.0" ixz="0.0" iyy="0.0001" iyz="0.0" izz="0.0001"/>
+    </inertial>
+  </link>
+  <joint name="imu_joint" type="fixed">
+    <origin xyz="-0.065 0 0.075" rpy="0 0 0" />
+    <parent link="base_link" />
+    <child link="imu_link" />
+  </joint>
+  <gazebo reference="imu_link">
+    <gravity>true</gravity>
+    <sensor name="imu_sensor" type="imu">
+      <always_on>true</always_on>
+      <update_rate>100</update_rate>
+      <visualize>true</visualize>
+      <plugin filename="libgazebo_ros_imu_sensor.so" name="imu_plugin">
+	<topicName>/ackermann_vehicle/imu</topicName>
+        <bodyName>imu_link</bodyName>
+        <updateRateHZ>100.0</updateRateHZ>
+        <gaussianNoise>0.0</gaussianNoise>
+        <xyzOffset>0 0 0</xyzOffset>
+        <rpyOffset>0 0 0</rpyOffset>
+        <frameName>imu_link</frameName>
+        <initialOrientationAsReference>false</initialOrientationAsReference>
+      </plugin>
+      <pose>0 0 0 0 0 0</pose>
+    </sensor>
+  </gazebo>
 </robot>

Commit message: Added automation code for testing

File: ackermann_vehicle_description/urdf/em_3905_hokuyo_imu.urdf.xacro (robot description, xacro)
@@ -357,24 +357,4 @@
   <xacro:rear_wheel lr_prefix="right" fr_prefix="rear"
                     lr_reflect="-1" fr_reflect="-1"/>
-  <!-- LiDAR -->
-  <!-- <link name="hokuyo_link">
-    <visual>
-      <geometry>
-        <box size="0.02 0.035 0.002"/>
-      </geometry>
-      <material name="Green"/>
-    </visual>
-    <inertial>
-      <mass value="0.001"/>
-      <origin xyz="0 0 0"/>
-      <inertia ixx="0.0001" ixy="0.0" ixz="0.0" iyy="0.0001" iyz="0.0" izz="0.0001"/>
-    </inertial>
-  </link>
-  <joint name="laser_joint" type="fixed">
-    <origin xyz="-0.065 0 0.075" rpy="0 0 0" />
-    <parent link="base_link" />
-    <child link="hokuyo_link" />
-  </joint>
--->
   <gazebo>
     <plugin name="gazebo_ros_control" filename="libgazebo_ros_control.so"/>
@@ -405,8 +385,4 @@
           <noise>
             <type>gaussian</type>
-            <!-- Noise parameters based on published spec for Hokuyo laser
-                achieving "+-30mm" accuracy at range < 10m.  A mean of 0.0m and
-                stddev of 0.01m will put 99.7% of samples within 0.03m of the true
-                reading. -->
             <mean>0.0</mean>
             <stddev>0.01</stddev>
@@ -420,5 +396,5 @@
     </gazebo>
   </xacro:macro>
-  <xacro:hokuyo_laser/>
+  <!-- <xacro:hokuyo_laser/> -->
   <!-- IMU frame -->
   <link name="imu_link">
@@ -447,5 +423,5 @@
       <visualize>true</visualize>
       <plugin filename="libgazebo_ros_imu_sensor.so" name="imu_plugin">
-	<topicName>/ackermann_vehicle/imu</topicName>
+	      <topicName>/ackermann_vehicle/imu</topicName>
         <bodyName>imu_link</bodyName>
         <updateRateHZ>100.0</updateRateHZ>
